Commit message: update: robot_description WEEK4

File: urdf/mobile_base.xacro (robot description, xacro)
@@ -8,5 +8,8 @@
   <xacro:property name="wheel_track" value="0.35"/>
   <xacro:property name="caster_radius" value="0.025"/>
-  <!-- base_footprint: Gốc chiếu xuống mặt đất -->
+  <!-- Tâm hộp nằm trước trục bánh một khoảng axle_offset.
+       Gốc base_link đặt TRÊN TRỤC BÁNH (chuẩn robot vi sai) để pose odometry
+       đúng là pose của base_footprint. -->
+  <xacro:property name="axle_offset" value="${base_length / 4.0}"/>
   <link name="base_footprint"/>
   <joint name="base_joint" type="fixed">
@@ -15,8 +18,7 @@
     <origin xyz="0 0 ${wheel_radius}" rpy="0 0 0"/>
   </joint>
-  <!-- base_link: Khung xe chính -->
   <link name="base_link">
     <visual>
-      <origin xyz="0 0 ${base_height / 2.0}" rpy="0 0 0"/>
+      <origin xyz="${axle_offset} 0 ${base_height / 2.0}" rpy="0 0 0"/>
       <geometry>
         <box size="${base_length} ${base_width} ${base_height}"/>
@@ -25,5 +27,5 @@
     </visual>
     <collision>
-      <origin xyz="0 0 ${base_height / 2.0}" rpy="0 0 0"/>
+      <origin xyz="${axle_offset} 0 ${base_height / 2.0}" rpy="0 0 0"/>
       <geometry>
         <box size="${base_length} ${base_width} ${base_height}"/>
@@ -31,7 +33,6 @@
     </collision>
     <xacro:box_inertia m="5.0" l="${base_length}" w="${base_width}" h="${base_height}"
-                       xyz="0 0 ${base_height / 2.0}" rpy="0 0 0"/>
+                       xyz="${axle_offset} 0 ${base_height / 2.0}" rpy="0 0 0"/>
   </link>
-  <!-- Macro tạo bánh xe dẫn động (Continuous Joint) -->
   <xacro:macro name="wheel" params="prefix y_reflect">
     <link name="${prefix}_wheel_link">
@@ -44,7 +45,7 @@
       </visual>
       <collision>
-        <origin xyz="0 0 0" rpy="${pi / 2.0} 0 0"/>
+        <origin xyz="0 0 0" rpy="0 0 0"/>
         <geometry>
-          <cylinder radius="${wheel_radius}" length="${wheel_length}"/>
+          <sphere radius="${wheel_radius}"/>
         </geometry>
       </collision>
@@ -55,5 +56,6 @@
       <parent link="base_link"/>
       <child link="${prefix}_wheel_link"/>
-      <origin xyz="${-base_length / 4.0} ${y_reflect * (wheel_track / 2.0)} 0" rpy="0 0 0"/>
+      <!-- x = 0: trục bánh trùng gốc base_link -->
+      <origin xyz="0 ${y_reflect * (wheel_track / 2.0)} 0" rpy="0 0 0"/>
       <axis xyz="0 1 0"/>
     </joint>
@@ -61,5 +63,4 @@
   <xacro:wheel prefix="left" y_reflect="1"/>
   <xacro:wheel prefix="right" y_reflect="-1"/>
-  <!-- Caster Wheel (Bánh phụ đa hướng) -->
   <link name="caster_wheel_link">
     <visual>
@@ -81,5 +82,5 @@
     <parent link="base_link"/>
     <child link="caster_wheel_link"/>
-    <origin xyz="${base_length / 3.0} 0 ${-(wheel_radius - caster_radius)}" rpy="0 0 0"/>
+    <origin xyz="${base_length / 3.0 + axle_offset} 0 ${-(wheel_radius - caster_radius)}" rpy="0 0 0"/>
   </joint>
 </robot>

File: urdf/robot.urdf.xacro (robot description, xacro)
@@ -4,3 +4,4 @@
   <xacro:include filename="mobile_base.xacro"/>
   <xacro:include filename="sensors.xacro"/>
+  <xacro:include filename="gazebo.xacro"/>
 </robot>

File: urdf/sensors.xacro (robot description, xacro)
@@ -21,5 +21,5 @@
     <parent link="base_link"/>
     <child link="lidar_link"/>
-    <origin xyz="0.1 0 0.12" rpy="0 0 0"/>
+    <origin xyz="${0.1 + axle_offset} 0 0.12" rpy="0 0 0"/>
   </joint>
   <!-- IMU Frame -->
